Commit message: Update the UR launch files for UR alone or with the Gripper

File: abdo_ws/src/my_ur_driver/my_moveit_config/srdf/my_world.macro.srdf.xacro (robot description, xacro)
@@ -53,116 +53,4 @@
     <disable_collisions link1="${prefix}wrist_1_link" link2="${prefix}wrist_3_link" reason="Never" />
     <disable_collisions link1="${prefix}wrist_2_link" link2="${prefix}wrist_3_link" reason="Adjacent" />
-    <!-- <disable_collisions link1="robotiq_base_link" link2="robotiq_140_base_link" reason="Adjacent gripper links" />
-    <disable_collisions link1="left_inner_finger" link2="left_inner_finger_pad" reason="Finger self-collision" />
-    <disable_collisions link1="right_inner_finger" link2="right_inner_finger_pad" reason="Finger self-collision" />
-    <disable_collisions link1="left_outer_finger" link2="left_outer_finger_pad" reason="Finger self-collision" />
-    <disable_collisions link1="right_outer_finger" link2="right_outer_finger_pad" reason="Finger self-collision" />
-    <disable_collisions link1="left_inner_finger" link2="left_outer_finger" reason="Finger self-collision" />
-    <disable_collisions link1="right_inner_finger" link2="right_outer_finger" reason="Finger self-collision" /> -->
-    <!-- <disable_collisions link1="left_outer_knuckle" link2="right_outer_knuckle" reason="Finger self-collision2" />
-    <disable_collisions link1="left_inner_knuckle" link2="right_inner_knuckle" reason="Finger self-collision4" />
-    <disable_collisions link1="left_inner_finger" link2="right_inner_finger" reason="Finger self-collision3" />
-    <disable_collisions link1="left_outer_finger" link2="right_outer_finger" reason="Finger self-collision5" />
-    <disable_collisions link1="left_inner_finger_pad" link2="right_inner_finger_pad" reason="Finger self-collision" />
-    <disable_collisions link1="left_outer_finger_pad" link2="right_outer_finger_pad" reason="Finger self-collision" />
-    <disable_collisions link1="robotiq_140_base_link" link2="robotiq_base_link" reason="Finger self-collision" /> -->
-    <!-- <disable_collisions link1="${prefix}robotiq_base_link" link2="${prefix}robotiq_140_base_link" reason="Adjacent gripper links" />
-    <disable_collisions link1="${prefix}left_inner_finger" link2="${prefix}left_inner_finger_pad" reason="Finger self-collision" />
-    <disable_collisions link1="${prefix}right_inner_finger" link2="${prefix}right_inner_finger_pad" reason="Finger self-collision" />
-    <disable_collisions link1="${prefix}left_outer_finger" link2="${prefix}left_outer_knuckle" reason="Finger self-collision" />
-    <disable_collisions link1="${prefix}right_inner_knuckle" link2="${prefix}right_outer_knuckle" reason="Finger self-collision" /> -->
-    <!-- <disable_collisions link1="${prefix}left_inner_finger" link2="${prefix}left_outer_finger" reason="Finger self-collision" />
-    <disable_collisions link1="${prefix}right_inner_finger" link2="${prefix}right_outer_finger" reason="Finger self-collision" />
-    <disable_collisions link1="${prefix}left_outer_knuckle" link2="${prefix}right_outer_knuckle" reason="Knuckle self-collision" />
-    <disable_collisions link1="${prefix}left_inner_knuckle" link2="${prefix}right_inner_knuckle" reason="Knuckle self-collision" />
-    <disable_collisions link1="${prefix}left_finger_tip" link2="${prefix}right_finger_tip" reason="Finger tip self-collision" /> -->
-    <!-- <disable_collisions link1="robotiq_base_link" link2="robotiq_140_base_link" reason="Adjacent" />
-    <disable_collisions link1="left_inner_finger" link2="left_inner_finger_pad" reason="Finger self-collision" />
-    <disable_collisions link1="right_inner_finger" link2="right_inner_finger_pad" reason="Finger self-collision" />
-    <disable_collisions link1="left_outer_knuckle" link2="left_outer_finger" reason="Finger self-collision" />
-    <disable_collisions link1="right_outer_knuckle" link2="right_outer_finger" reason="Finger self-collision" />
-    <disable_collisions link1="tool0" link2="robotiq_base_link" reason="Adjacent" />
-    <disable_collisions link1="robotiq_base_link" link2="left_outer_knuckle" reason="Adjacent" />
-    <disable_collisions link1="robotiq_base_link" link2="right_outer_knuckle" reason="Adjacent" />
-    <disable_collisions link1="robotiq_base_link" link2="left_inner_knuckle" reason="Adjacent" />
-    <disable_collisions link1="robotiq_base_link" link2="right_inner_knuckle" reason="Adjacent" />
-    <disable_collisions link1="left_outer_finger" link2="left_inner_finger" reason="Finger self-collision" />
-    <disable_collisions link1="right_outer_finger" link2="right_inner_finger" reason="Finger self-collision" /> -->
-<!-- Base and Gripper Collisions -->
-    <disable_collisions link1="robotiq_base_link" link2="robotiq_140_base_link" reason="Adjacent" />
-    <disable_collisions link1="robotiq_base_link" link2="left_inner_finger" reason="Finger self-collision" />
-    <disable_collisions link1="robotiq_base_link" link2="left_inner_finger_pad" reason="Finger self-collision" />
-    <disable_collisions link1="robotiq_base_link" link2="left_outer_knuckle" reason="Adjacent" />
-    <disable_collisions link1="robotiq_base_link" link2="left_outer_finger" reason="Finger self-collision" />
-    <disable_collisions link1="robotiq_base_link" link2="right_inner_finger" reason="Finger self-collision" />
-    <disable_collisions link1="robotiq_base_link" link2="right_inner_finger_pad" reason="Finger self-collision" />
-    <disable_collisions link1="robotiq_base_link" link2="right_outer_knuckle" reason="Adjacent" />
-    <disable_collisions link1="robotiq_base_link" link2="right_outer_finger" reason="Finger self-collision" />
-    <disable_collisions link1="robotiq_base_link" link2="left_inner_knuckle" reason="Adjacent" />
-    <disable_collisions link1="robotiq_base_link" link2="right_inner_knuckle" reason="Adjacent" />
-    <disable_collisions link1="robotiq_140_base_link" link2="left_inner_finger" reason="Finger self-collision" />
-    <disable_collisions link1="robotiq_140_base_link" link2="left_inner_finger_pad" reason="Finger self-collision" />
-    <disable_collisions link1="robotiq_140_base_link" link2="left_outer_knuckle" reason="Finger self-collision" />
-    <disable_collisions link1="robotiq_140_base_link" link2="left_outer_finger" reason="Finger self-collision" />
-    <disable_collisions link1="robotiq_140_base_link" link2="right_inner_finger" reason="Finger self-collision" />
-    <disable_collisions link1="robotiq_140_base_link" link2="right_inner_finger_pad" reason="Finger self-collision" />
-    <disable_collisions link1="robotiq_140_base_link" link2="right_outer_knuckle" reason="Finger self-collision" />
-    <disable_collisions link1="robotiq_140_base_link" link2="right_outer_finger" reason="Finger self-collision" />
-    <disable_collisions link1="robotiq_140_base_link" link2="left_inner_knuckle" reason="Finger self-collision" />
-    <disable_collisions link1="robotiq_140_base_link" link2="right_inner_knuckle" reason="Finger self-collision" />
-    <disable_collisions link1="left_inner_finger" link2="left_inner_finger_pad" reason="Finger self-collision" />
-    <disable_collisions link1="left_inner_finger" link2="left_outer_knuckle" reason="Finger self-collision" />
-    <disable_collisions link1="left_inner_finger" link2="left_outer_finger" reason="Finger self-collision" />
-    <disable_collisions link1="left_inner_finger" link2="right_inner_finger" reason="Finger self-collision" />
-    <disable_collisions link1="left_inner_finger" link2="right_inner_finger_pad" reason="Finger self-collision" />
-    <disable_collisions link1="left_inner_finger" link2="right_outer_knuckle" reason="Finger self-collision" />
-    <disable_collisions link1="left_inner_finger" link2="right_outer_finger" reason="Finger self-collision" />
-    <disable_collisions link1="left_inner_finger" link2="left_inner_knuckle" reason="Finger self-collision" />
-    <disable_collisions link1="left_inner_finger" link2="right_inner_knuckle" reason="Finger self-collision" />
-    <disable_collisions link1="left_inner_finger_pad" link2="left_outer_knuckle" reason="Finger self-collision" />
-    <disable_collisions link1="left_inner_finger_pad" link2="left_outer_finger" reason="Finger self-collision" />
-    <disable_collisions link1="left_inner_finger_pad" link2="right_inner_finger" reason="Finger self-collision" />
-    <disable_collisions link1="left_inner_finger_pad" link2="right_inner_finger_pad" reason="Finger self-collision" />
-    <disable_collisions link1="left_inner_finger_pad" link2="right_outer_knuckle" reason="Finger self-collision" />
-    <disable_collisions link1="left_inner_finger_pad" link2="right_outer_finger" reason="Finger self-collision" />
-    <disable_collisions link1="left_inner_finger_pad" link2="left_inner_knuckle" reason="Finger self-collision" />
-    <disable_collisions link1="left_inner_finger_pad" link2="right_inner_knuckle" reason="Finger self-collision" />
-    <disable_collisions link1="left_outer_knuckle" link2="left_outer_finger" reason="Finger self-collision" />
-    <disable_collisions link1="left_outer_knuckle" link2="right_inner_finger" reason="Finger self-collision" />
-    <disable_collisions link1="left_outer_knuckle" link2="right_inner_finger_pad" reason="Finger self-collision" />
-    <disable_collisions link1="left_outer_knuckle" link2="right_outer_knuckle" reason="Finger self-collision" />
-    <disable_collisions link1="left_outer_knuckle" link2="right_outer_finger" reason="Finger self-collision" />
-    <disable_collisions link1="left_outer_knuckle" link2="left_inner_knuckle" reason="Finger self-collision" />
-    <disable_collisions link1="left_outer_knuckle" link2="right_inner_knuckle" reason="Finger self-collision" />
-    <disable_collisions link1="left_outer_finger" link2="right_inner_finger" reason="Finger self-collision" />
-    <disable_collisions link1="left_outer_finger" link2="right_inner_finger_pad" reason="Finger self-collision" />
-    <disable_collisions link1="left_outer_finger" link2="right_outer_knuckle" reason="Finger self-collision" />
-    <disable_collisions link1="left_outer_finger" link2="right_outer_finger" reason="Finger self-collision" />
-    <disable_collisions link1="left_outer_finger" link2="left_inner_knuckle" reason="Finger self-collision" />
-    <disable_collisions link1="left_outer_finger" link2="right_inner_knuckle" reason="Finger self-collision" />
-    <disable_collisions link1="right_inner_finger" link2="right_inner_finger_pad" reason="Finger self-collision" />
-    <disable_collisions link1="right_inner_finger" link2="right_outer_knuckle" reason="Finger self-collision" />
-    <disable_collisions link1="right_inner_finger" link2="right_outer_finger" reason="Finger self-collision" />
-    <disable_collisions link1="right_inner_finger" link2="left_inner_knuckle" reason="Finger self-collision" />
-    <disable_collisions link1="right_inner_finger" link2="right_inner_knuckle" reason="Finger self-collision" />
-    <disable_collisions link1="right_inner_finger_pad" link2="right_outer_knuckle" reason="Finger self-collision" />
-    <disable_collisions link1="right_inner_finger_pad" link2="right_outer_finger" reason="Finger self-collision" />
-    <disable_collisions link1="right_inner_finger_pad" link2="left_inner_knuckle" reason="Finger self-collision" />
-    <disable_collisions link1="right_inner_finger_pad" link2="right_inner_knuckle" reason="Finger self-collision" />
-    <disable_collisions link1="right_outer_knuckle" link2="right_outer_finger" reason="Finger self-collision" />
-    <disable_collisions link1="right_outer_knuckle" link2="left_inner_knuckle" reason="Finger self-collision" />
-    <disable_collisions link1="right_outer_knuckle" link2="right_inner_knuckle" reason="Finger self-collision" />
-    <disable_collisions link1="right_outer_finger" link2="left_inner_knuckle" reason="Finger self-collision" />
-    <disable_collisions link1="right_outer_finger" link2="right_inner_knuckle" reason="Finger self-collision" />
-    <disable_collisions link1="left_inner_knuckle" link2="right_inner_knuckle" reason="Finger self-collision" />
-    <disable_collisions link1="robotiq_base_link" link2="robotiq_140_base_link" reason="Adjacent" />
-    <disable_collisions link1="robotiq_base_link" link2="tool0" reason="Adjacent" />
-    <disable_collisions link1="robotiq_base_link" link2="wrist_1_link" reason="Adjacent" />
-    <disable_collisions link1="robotiq_base_link" link2="wrist_2_link" reason="Adjacent" />
-    <disable_collisions link1="robotiq_base_link" link2="wrist_3_link" reason="Adjacent" />
-    <disable_collisions link1="robotiq_140_base_link" link2="tool0" reason="Adjacent" />
-    <disable_collisions link1="robotiq_140_base_link" link2="wrist_1_link" reason="Adjacent" />
-    <disable_collisions link1="robotiq_140_base_link" link2="wrist_2_link" reason="Adjacent" />
-    <disable_collisions link1="robotiq_140_base_link" link2="wrist_3_link" reason="Adjacent" />
     <disable_collisions link1="tool0" link2="wrist_1_link" reason="Adjacent" />
     <disable_collisions link1="tool0" link2="wrist_2_link" reason="Adjacent" />
@@ -184,5 +72,4 @@
     <disable_collisions link1="tool0_2_cam_holder_with_onrobot_single" link2="wrist_3_link" reason="Adjacent" />
  -->
-cam_holder_with_onrobot_single
   </xacro:macro>
 </robot>

File: abdo_ws/src/my_ur_driver/my_ur_config/urdf/my world.urdf.xacro (robot description, xacro)
@@ -5,7 +5,4 @@
    <!-- import main macro -->
    <xacro:include filename="$(find ur_description)/urdf/ur_macro.xacro"/>
-   <xacro:include filename="$(find my_ur_driver)/urdf/robotiq_2f_140.xacro" />
-   <xacro:include filename="$(find my_ur_driver)/urdf/robotiq_2f_140_gripper.urdf.xacro" />
-   <xacro:include filename="$(find my_ur_driver)/urdf/2f_140.ros2_control.xacro" />
    <!-- possible 'ur_type' values: ur3, ur3e, ur5, ur5e, ur10, ur10e, ur16e, ur20, ur30 -->
    <!-- the default value should raise an error in case this was called without defining the type -->
@@ -163,10 +160,4 @@
     <origin xyz="0 0 0" rpy="0 0 0" />
   </joint>
-  <link name="robotiq_2f_140" />
-  <joint name="robotiq_2f_140_" type="fixed">
-    <parent link="tool0" />
-    <child link="robotiq_2f_140" />
-    <origin xyz="0 0 0.205" rpy="0 0 0" />
-  </joint>
     <!-- this part deals with the tcp end effector transform, not related to the visual/collision. -->
   <!-- so far tcp_gripper is always required even if u dun use it, because the my_robot_advance.cpp always look for it at the start -->

Commit message: Update the urdf to include urdf for UR only or with gripper

File: abdo_ws/src/my_ur_driver/my_moveit_config/srdf/my_world.macro.srdf.xacro (robot description, xacro)
@@ -59,17 +59,4 @@
     <disable_collisions link1="wrist_1_link" link2="wrist_3_link" reason="Adjacent" />
     <disable_collisions link1="wrist_2_link" link2="wrist_3_link" reason="Adjacent" />
-    <disable_collisions link1="cam_holder_with_onrobot_single" link2="robotiq_base_link" reason="Adjacent" />
-    <disable_collisions link1="cam_holder_with_onrobot_single" link2="robotiq_140_base_link" reason="Adjacent" />
-    <disable_collisions link1="cam_holder_with_onrobot_single" link2="tool0" reason="Adjacent" />
-    <disable_collisions link1="cam_holder_with_onrobot_single" link2="wrist_1_link" reason="Adjacent" />
-    <disable_collisions link1="cam_holder_with_onrobot_single" link2="wrist_2_link" reason="Adjacent" />
-    <disable_collisions link1="cam_holder_with_onrobot_single" link2="wrist_3_link" reason="Adjacent" />
-    <!-- <disable_collisions link1="tool0_2_cam_holder_with_onrobot_single" link2="robotiq_base_link" reason="Adjacent" />
-    <disable_collisions link1="tool0_2_cam_holder_with_onrobot_single" link2="robotiq_140_base_link" reason="Adjacent" />
-    <disable_collisions link1="tool0_2_cam_holder_with_onrobot_single" link2="tool0" reason="Adjacent" />
-    <disable_collisions link1="tool0_2_cam_holder_with_onrobot_single" link2="wrist_1_link" reason="Adjacent" />
-    <disable_collisions link1="tool0_2_cam_holder_with_onrobot_single" link2="wrist_2_link" reason="Adjacent" />
-    <disable_collisions link1="tool0_2_cam_holder_with_onrobot_single" link2="wrist_3_link" reason="Adjacent" />
- -->
   </xacro:macro>
 </robot>

File: abdo_ws/src/my_ur_driver/my_ur_config/urdf/my_world.urdf.xacro (robot description, xacro)
@@ -7,5 +7,5 @@
    <!-- possible 'ur_type' values: ur3, ur3e, ur5, ur5e, ur10, ur10e, ur16e, ur20, ur30 -->
    <!-- the default value should raise an error in case this was called without defining the type -->
-   <xacro:arg name="ur_type" default="ur5x"/>
+   <xacro:arg name="ur_type" default="ur10e"/>
    <!-- parameters -->
    <xacro:arg name="tf_prefix" default="" />
@@ -50,5 +50,5 @@
    <xacro:property name="initial_positions_file" default="$(arg initial_positions_file)"/>
    <!-- create link fixed to the "world" -->
-   <!-- <link name="world" /> -->
+   <link name="world" />
    <!-- arm -->
    <xacro:ur_robot

File: abdo_ws/src/my_ur_driver/my_ur_config/urdf/my_world_with_gripper.urdf.xacro (robot description, xacro)
@@ -11,5 +11,5 @@
    <!-- possible 'ur_type' values: ur3, ur3e, ur5, ur5e, ur10, ur10e, ur16e, ur20, ur30 -->
    <!-- the default value should raise an error in case this was called without defining the type -->
-   <xacro:arg name="ur_type" default="ur5x"/>
+   <xacro:arg name="ur_type" default="ur10e"/>
    <!-- parameters -->
    <xacro:arg name="tf_prefix" default="" />
